File: jomox_resonator_multi_fx_modboard/jomox_resonator_multi_fx_modboard.kicad_pcb (KiCad board)
At the start: 2 copper layers, 27.7 x 19.8 mm, 14 parts, among them J1 Bank_Up, J2 Bank_Down, J3 ISP, U1 24LC32, U2 24LC32, U3 ATtiny85-20S

Commit message: finalized modboard design
Parts:
- removed J1: Bank_Up, Connector_PinHeader_2.54mm:PinHeader_1x02_P2.54mm_Vertical
- removed J2: Bank_Down, Connector_PinHeader_2.54mm:PinHeader_1x02_P2.54mm_Vertical
- added J4: Conn, Connector_PinHeader_2.54mm:PinHeader_1x04_P2.54mm_Vertical, F.Cu at (73.5, 46.8)
- moved R3 20.5 mm to (72.7, 59.4), turned to 180 degrees
- moved C2 18.2 mm to (69.2, 47.2)
- moved J3 18.2 mm to (65.7, 57.5)
- moved C1 18.2 mm to (64.4, 52.5)
- moved NT1 18.2 mm to (64.4, 58.5)
- moved NT2 18.2 mm to (65.7, 58.5)
- moved NT3 18.2 mm to (65.7, 56.5)
- moved R1 18.2 mm to (64.3, 54.5)
- moved U1 18.2 mm to (50.0, 50.2)
- moved U2 18.2 mm to (65.5, 49.1)
- moved U3 18.2 mm to (64.9, 48.5)
- moved R2 17.6 mm to (72.7, 57.3), turned to 180 degrees
Connections:
- R2 pad 1: +3V3 -> /Bank_Down
- R2 pad 2: /Bank_Down -> +3V3
- R3 pad 1: +3V3 -> /Bank_Up
- R3 pad 2: /Bank_Up -> +3V3
- U1 pad 7: /WP -> unconnected-(U1-WP-Pad7)
Routing:
- net /WP: track 40.4 -> 28.5 mm
- net GND: track 27.8 -> 22.9 mm
- net /Bank_Down: track 9.32 -> 13.0 mm
- net /Bank_Up: track 13.7 -> 17.4 mm
- net +3V3: track 48.6 -> 51.8 mm
- net /SCL: track 35.5 -> 35.0 mm, vias 3 -> 2
Other:
- board size 27.7 x 19.8 mm -> 27.7 x 19.9 mm
- board text added: "Jomox Resonator Multi FX Modboard v0.2"
- board text removed: "Jomox Resonator Multi FX Modboard v0.1"
